File: Dyno_Harness_2026_KiCad/Components.kicad_sch (KiCad schematic)
At the start: 44 parts, among them P1 Fuel Pump, SW1 Upshift, SW2 downshift, T1 Clutch DC/DC Converter, U1 IAT + MAP

Commit message: Did DRC and ERC for all schematics and layouts
Parts:
- Camshaft Position1: renamed from Camshaft Position
- Coolant Temp1: renamed from Coolant Temp
- Crankshaft Pos1: renamed from Crankshaft Pos
- MoTeC LTCDB1: renamed from MoTeC LTCDB
- Oil Pressure1: renamed from Oil Pressure
- Oil Temperature1: renamed from Oil Temperature
- Starter Switch1: renamed from Starter Switch
- gave numbers to parts that had none: 4
- renumbered BATTERY to BATTERY1, DASH_ETH to DASH_ETH1, ECU_ETH to ECU_ETH1, EPS to EPS1, FP to FP1, IGN to IGN1, MS to MS1, RPS to RPS1, RS to RS1, SM to SM3, TB to TB1
