File: Dyno_Harness_2026_KiCad/PDM15.kicad_sch (KiCad schematic)
At the start: 3 parts, among them J3 PDM15/30 Connector A - MoTeC, J4 PDM15/30 Connector B - MoTeC

Commit message: Did DRC and ERC for all schematics and layouts
Parts:
- PDM15/30 Connector C1: renamed from PDM15/30 Connector C
Changed lines of the file:
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@@
 		(in_pos_files yes)
 		(dnp no)
-		(property "Reference" "PDM15/30 Connector C"
+		(property "Reference" "PDM15/30 Connector C1"
 			(at 305.308 107.95 90)
 			(show_name no)
@@
 			(project "Dyno Harness 2026"
 				(path "/01d52fff-0621-4906-b716-923629de591a"
-					(reference "PDM15/30 Connector C")
+					(reference "PDM15/30 Connector C1")
 					(unit 1)
 				)
