File: Strain_Gauge_Alternate_KiCad/Strain Gauge Alternate.kicad_sch (KiCad schematic)
At the start: 13 parts, among them J1 SSW-103-01-G-S, J2 SSW-103-01-G-S, U1 INA121PA, U2 UA741CP

Commit message: Did DRC and ERC for all schematics and layouts
Changed lines of the file:
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@@
 		(in_pos_files yes)
 		(dnp no)
-		(property "Reference" "#PWR?"
+		(property "Reference" "#PWR03"
 			(at 63.5 83.82 0)
 			(hide yes)
@@
 			(project "Strain Gauge Alternate"
 				(path "/67086dc8-797e-49ef-8e82-194f9c4e0532"
-					(reference "#PWR?")
+					(reference "#PWR03")
 					(unit 1)
 				)
@@
 		(in_pos_files yes)
 		(dnp no)
-		(property "Reference" "#PWR?"
+		(property "Reference" "#PWR07"
 			(at 134.62 83.82 0)
 			(hide yes)
@@
 			(project "Strain Gauge Alternate"
 				(path "/67086dc8-797e-49ef-8e82-194f9c4e0532"
-					(reference "#PWR?")
+					(reference "#PWR07")
 					(unit 1)
 				)
@@
 		(dnp no)
 		(property "Reference" "ST4"
-			(at 68.58 152.4 90)
+			(at 69.342 150.622 90)
 			(show_name no)
 			(do_not_autoplace no)
@@
 		)
 		(property "Value" "PTH-M2D5X5"
-			(at 66.04 149.86 90)
+			(at 66.802 148.082 90)
 			(show_name no)
 			(do_not_autoplace no)
@@
 		(in_pos_files yes)
 		(dnp no)
-		(property "Reference" "#PWR?"
+		(property "Reference" "#PWR06"
 			(at 71.12 160.02 0)
 			(hide yes)
@@
 			(project "Strain Gauge Alternate"
 				(path "/67086dc8-797e-49ef-8e82-194f9c4e0532"
-					(reference "#PWR?")
+					(reference "#PWR06")
 					(unit 1)
 				)
@@
 		(in_pos_files yes)
 		(dnp no)
-		(property "Reference" "#PWR?"
+		(property "Reference" "#PWR09"
 			(at 139.7 124.46 0)
 			(hide yes)
@@
 			(project "Strain Gauge Alternate"
 				(path "/67086dc8-797e-49ef-8e82-194f9c4e0532"
-					(reference "#PWR?")
+					(reference "#PWR09")
 					(unit 1)
 				)
@@
 		(in_pos_files yes)
 		(dnp no)
-		(property "Reference" "#PWR?"
+		(property "Reference" "#PWR011"
 			(at 170.18 129.54 0)
 			(hide yes)
@@
 			(project "Strain Gauge Alternate"
 				(path "/67086dc8-797e-49ef-8e82-194f9c4e0532"
-					(reference "#PWR?")
+					(reference "#PWR011")
 					(unit 1)
 				)
@@
 		(dnp no)
 		(property "Reference" "ST2"
-			(at 68.58 129.54 90)
+			(at 69.342 127.762 90)
 			(show_name no)
 			(do_not_autoplace no)
@@
 		)
 		(property "Value" "PTH-M2D5X5"
-			(at 66.04 127 90)
+			(at 66.802 125.222 90)
 			(show_name no)
 			(do_not_autoplace no)
@@
 		(dnp no)
 		(property "Reference" "ST3"
-			(at 50.8 152.4 90)
+			(at 51.562 150.622 90)
 			(show_name no)
 			(do_not_autoplace no)
@@
 		)
 		(property "Value" "PTH-M2D5X5"
-			(at 48.26 149.86 90)
+			(at 49.022 148.082 90)
 			(show_name no)
 			(do_not_autoplace no)
@@
 		(in_pos_files yes)
 		(dnp no)
-		(property "Reference" "#PWR?"
+		(property "Reference" "#PWR010"
 			(at 139.7 149.86 0)
 			(hide yes)
@@
 			(project "Strain Gauge Alternate"
 				(path "/67086dc8-797e-49ef-8e82-194f9c4e0532"
-					(reference "#PWR?")
+					(reference "#PWR010")
 					(unit 1)
 				)
@@
 		(dnp no)
 		(property "Reference" "ST1"
-			(at 50.8 129.54 90)
+			(at 51.562 127.762 90)
 			(show_name no)
 			(do_not_autoplace no)
@@
 		)
 		(property "Value" "PTH-M2D5X5"
-			(at 48.26 127 90)
+			(at 49.022 125.222 90)
 			(show_name no)
 			(do_not_autoplace no)
@@
 		(in_pos_files yes)
 		(dnp no)
-		(property "Reference" "#PWR?"
+		(property "Reference" "#PWR04"
 			(at 63.5 109.22 0)
 			(hide yes)
@@
 			(project "Strain Gauge Alternate"
 				(path "/67086dc8-797e-49ef-8e82-194f9c4e0532"
-					(reference "#PWR?")
+					(reference "#PWR04")
 					(unit 1)
 				)
@@
 		(in_pos_files yes)
 		(dnp no)
-		(property "Reference" "#PWR?"
+		(property "Reference" "#PWR02"
 			(at 53.34 160.02 0)
 			(hide yes)
@@
 			(project "Strain Gauge Alternate"
 				(path "/67086dc8-797e-49ef-8e82-194f9c4e0532"
-					(reference "#PWR?")
+					(reference "#PWR02")
 					(unit 1)
 				)
@@
 		(in_pos_files yes)
 		(dnp no)
-		(property "Reference" "#PWR?"
+		(property "Reference" "#PWR08"
 			(at 134.62 104.14 0)
 			(hide yes)
@@
 			(project "Strain Gauge Alternate"
 				(path "/67086dc8-797e-49ef-8e82-194f9c4e0532"
-					(reference "#PWR?")
+					(reference "#PWR08")
 					(unit 1)
 				)
@@
 		(in_pos_files yes)
 		(dnp no)
-		(property "Reference" "#PWR?"
+		(property "Reference" "#PWR05"
 			(at 71.12 137.16 0)
 			(hide yes)
@@
 			(project "Strain Gauge Alternate"
 				(path "/67086dc8-797e-49ef-8e82-194f9c4e0532"
-					(reference "#PWR?")
+					(reference "#PWR05")
 					(unit 1)
 				)
@@
 		(in_pos_files yes)
 		(dnp no)
-		(property "Reference" "#PWR?"
+		(property "Reference" "#PWR012"
 			(at 170.18 149.86 0)
 			(hide yes)
@@
 			(project "Strain Gauge Alternate"
 				(path "/67086dc8-797e-49ef-8e82-194f9c4e0532"
-					(reference "#PWR?")
+					(reference "#PWR012")
 					(unit 1)
 				)
@@
 		(in_pos_files yes)
 		(dnp no)
-		(property "Reference" "#PWR?"
+		(property "Reference" "#PWR01"
 			(at 53.34 137.16 0)
 			(hide yes)
@@
 			(project "Strain Gauge Alternate"
 				(path "/67086dc8-797e-49ef-8e82-194f9c4e0532"
-					(reference "#PWR?")
+					(reference "#PWR01")
 					(unit 1)
 				)
